Commit message: Added a neck to Hubo.

File: public/hubo-urdf/model.urdf (robot description, URDF)
Before this commit: robot huboplus, 57 links, 56 joints
Links:
- added link Body_HNR
- added link Body_HNY; collision mesh filename=./meshes/Body_HNY_col.dae
Joints:
- added joint HNR: type revolute, parent Body_HNY, child Body_HNR, origin xyz=-0.0014665 0.0024526 0.0876725 rpy=0 -0 0, axis 1 0 0, limit lower=-0.523599 upper=0.523599 effort=10.0 velocity=1.0
- added joint HNY: type revolute, parent Body_Torso, child Body_HNY, origin xyz=0.0137246 0.0 0.1092625 rpy=0 -0 0, axis 0 0 1, limit lower=-1.5 upper=1.5 effort=10.0 velocity=1.0
- joint HNP: origin xyz=0.0122581 0.0024526 0.196935 rpy=0 -0 0 -> xyz=0 0 0 rpy=0 -0 0; parent Body_Torso -> Body_HNR

Commit message: Got fingers working. Invented a Hubo.coffee class in order to implement finger functionality.

File: public/hubo-urdf/model.urdf (robot description, URDF)
Before this commit: robot huboplus, 59 links, 58 joints
Joints:
- removed joint Knuckle2
- removed joint Knuckle212
- removed joint Knuckle215
- removed joint Knuckle218
- removed joint Knuckle221
- removed joint Knuckle230
- removed joint Knuckle233
- removed joint Knuckle236
- removed joint Knuckle239
- removed joint Knuckle29
- removed joint Knuckle3
- removed joint Knuckle310
- removed joint Knuckle313
- removed joint Knuckle316
- removed joint Knuckle319
- removed joint Knuckle322
- removed joint Knuckle331
- removed joint Knuckle334
- removed joint Knuckle337
- removed joint Knuckle340
- added joint leftIndexKnuckle2: type revolute, parent leftIndexProximal, child leftIndexMedial, origin xyz=0.032 0 0 rpy=0 -0 0, axis 0 0 -1, limit lower=-3.14 upper=3.14 effort=10.0 velocity=1.0
- added joint leftIndexKnuckle3: type revolute, parent leftIndexMedial, child leftIndexDistal, origin xyz=0.022 0 0 rpy=0 -0 0, axis 0 0 -1, limit lower=-3.14 upper=3.14 effort=10.0 velocity=1.0
- added joint leftMiddleKnuckle2: type revolute, parent leftMiddleProximal, child leftMiddleMedial, origin xyz=0.032 0 0 rpy=0 -0 0, axis 0 0 -1, limit lower=-3.14 upper=3.14 effort=10.0 velocity=1.0
- added joint leftMiddleKnuckle3: type revolute, parent leftMiddleMedial, child leftMiddleDistal, origin xyz=0.022 0 0 rpy=0 -0 0, axis 0 0 -1, limit lower=-3.14 upper=3.14 effort=10.0 velocity=1.0
- added joint leftPinkyKnuckle2: type revolute, parent leftPinkyProximal, child leftPinkyMedial, origin xyz=0.032 0 0 rpy=0 -0 0, axis 0 0 -1, limit lower=-3.14 upper=3.14 effort=10.0 velocity=1.0
- added joint leftPinkyKnuckle3: type revolute, parent leftPinkyMedial, child leftPinkyDistal, origin xyz=0.022 0 0 rpy=0 -0 0, axis 0 0 -1, limit lower=-3.14 upper=3.14 effort=10.0 velocity=1.0
- added joint leftRingKnuckle2: type revolute, parent leftRingProximal, child leftRingMedial, origin xyz=0.032 0 0 rpy=0 -0 0, axis 0 0 -1, limit lower=-3.14 upper=3.14 effort=10.0 velocity=1.0
- added joint leftRingKnuckle3: type revolute, parent leftRingMedial, child leftRingDistal, origin xyz=0.022 0 0 rpy=0 -0 0, axis 0 0 -1, limit lower=-3.14 upper=3.14 effort=10.0 velocity=1.0
- added joint leftThumbKnuckle2: type revolute, parent leftThumbProximal, child leftThumbMedial, origin xyz=0.032 0 0 rpy=0 -0 0, axis 0 0 -1, limit lower=-3.14 upper=3.14 effort=10.0 velocity=1.0
- added joint leftThumbKnuckle3: type revolute, parent leftThumbMedial, child leftThumbDistal, origin xyz=0.022 0 0 rpy=0 -0 0, axis 0 0 -1, limit lower=-3.14 upper=3.14 effort=10.0 velocity=1.0
- added joint rightIndexKnuckle2: type revolute, parent rightIndexProximal, child rightIndexMedial, origin xyz=0.032 0 0 rpy=0 -0 0, axis 0 0 -1, limit lower=0 upper=1.57 effort=10.0 velocity=1.0
- added joint rightIndexKnuckle3: type revolute, parent rightIndexMedial, child rightIndexDistal, origin xyz=0.022 0 0 rpy=0 -0 0, axis 0 0 -1, limit lower=0 upper=1.57 effort=10.0 velocity=1.0
- added joint rightMiddleKnuckle2: type revolute, parent rightMiddleProximal, child rightMiddleMedial, origin xyz=0.032 0 0 rpy=0 -0 0, axis 0 0 -1, limit lower=0 upper=1.57 effort=10.0 velocity=1.0
- added joint rightMiddleKnuckle3: type revolute, parent rightMiddleMedial, child rightMiddleDistal, origin xyz=0.022 0 0 rpy=0 -0 0, axis 0 0 -1, limit lower=0 upper=1.57 effort=10.0 velocity=1.0
- added joint rightPinkyKnuckle2: type revolute, parent rightPinkyProximal, child rightPinkyMedial, origin xyz=0.032 0 0 rpy=0 -0 0, axis 0 0 -1, limit lower=0 upper=1.57 effort=10.0 velocity=1.0
- added joint rightPinkyKnuckle3: type revolute, parent rightPinkyMedial, child rightPinkyDistal, origin xyz=0.022 0 0 rpy=0 -0 0, axis 0 0 -1, limit lower=0 upper=1.57 effort=10.0 velocity=1.0
- added joint rightRingKnuckle2: type revolute, parent rightRingProximal, child rightRingMedial, origin xyz=0.032 0 0 rpy=0 -0 0, axis 0 0 -1, limit lower=0 upper=1.57 effort=10.0 velocity=1.0
- added joint rightRingKnuckle3: type revolute, parent rightRingMedial, child rightRingDistal, origin xyz=0.022 0 0 rpy=0 -0 0, axis 0 0 -1, limit lower=0 upper=1.57 effort=10.0 velocity=1.0
- added joint rightThumbKnuckle2: type revolute, parent rightThumbProximal, child rightThumbMedial, origin xyz=0.032 0 0 rpy=0 -0 0, axis 0 0 -1, limit lower=0 upper=1.57 effort=10.0 velocity=1.0
- added joint rightThumbKnuckle3: type revolute, parent rightThumbMedial, child rightThumbDistal, origin xyz=0.022 0 0 rpy=0 -0 0, axis 0 0 -1, limit lower=0 upper=1.57 effort=10.0 velocity=1.0
- joint leftIndexKnuckle1: axis 0 0 1 -> 0 0 -1
- joint leftMiddleKnuckle1: axis 0 0 1 -> 0 0 -1
- joint leftPinkyKnuckle1: axis 0 0 1 -> 0 0 -1
- joint leftRingKnuckle1: axis 0 0 1 -> 0 0 -1
- joint leftThumbKnuckle1: axis 0 0 1 -> 0 0 -1
- joint rightIndexKnuckle1: axis 0 0 1 -> 0 0 -1; limit lower=-3.14 upper=3.14 effort=10.0 velocity=1.0 -> lower=0 upper=1.57 effort=10.0 velocity=1.0
- joint rightMiddleKnuckle1: axis 0 0 1 -> 0 0 -1; limit lower=-3.14 upper=3.14 effort=10.0 velocity=1.0 -> lower=0 upper=1.57 effort=10.0 velocity=1.0
- joint rightPinkyKnuckle1: axis 0 0 1 -> 0 0 -1; limit lower=-3.14 upper=3.14 effort=10.0 velocity=1.0 -> lower=0 upper=1.57 effort=10.0 velocity=1.0
- joint rightRingKnuckle1: axis 0 0 1 -> 0 0 -1; limit lower=-3.14 upper=3.14 effort=10.0 velocity=1.0 -> lower=0 upper=1.57 effort=10.0 velocity=1.0
- joint rightThumbKnuckle1: axis 0 0 1 -> 0 0 -1; limit lower=-3.14 upper=3.14 effort=10.0 velocity=1.0 -> lower=0 upper=1.57 effort=10.0 velocity=1.0

Commit message: Fixed the neck kinematics, cause they were wrong before.

File: public/hubo-urdf/model.urdf (robot description, URDF)
Before this commit: robot huboplus, 59 links, 58 joints
Links:
- removed link Body_HNP
- removed link Body_HNR
- removed link Body_HNY
- added link Body_Head, mass 0.374251; collision mesh filename=./meshes/Body_Head_col.dae; visual mesh filename=./meshes/Body_Head_vis.dae
- added link Body_Head_Empty
- added link Body_Neck; collision mesh filename=./meshes/Body_Neck_col.dae
Joints:
- joint HNP: child Body_HNP -> Body_Head_Empty; parent Body_HNR -> Body_Neck
- joint HNR: child Body_HNR -> Body_Head; parent Body_HNY -> Body_Head_Empty
- joint HNY: child Body_HNY -> Body_Neck

Commit message: More improvements to trajectory_playback.jade BUT I have disable NK1 and NK2 for now.

File: public/hubo-urdf/model.urdf (robot description, URDF)
Before this commit: robot huboplus, 59 links, 58 joints
Joints:
- removed joint HNY
- added joint NKY: type revolute, parent Body_Torso, child Body_Neck, origin xyz=0.0137246 0.0 0.1092625 rpy=0 -0 0, axis 0 0 1, limit lower=-1.5 upper=1.5 effort=10.0 velocity=1.0

Commit message: Made stuff more robust. Fixed WST joint. Increased FPS. Almost ready for demo.

File: public/hubo-urdf/model.urdf (robot description, URDF)
Before this commit: robot huboplus, 59 links, 58 joints
Joints:
- removed joint HPY
- added joint WST: type revolute, parent Body_Torso, child Body_Hip, origin xyz=0.0122662 0.00245974 -0.15262 rpy=0 -0 0, axis 0 0 -1, limit lower=-3.14158 upper=3.14158 effort=10.0 velocity=1.0
