Commit message: Added hubo-urdf as submodule. Also, added updated /out files forgotten in moving hubo-trajectories to a submodule.

File: out/data/hubo-urdf/model.urdf (robot description, URDF)
Before this commit: robot huboplus, 59 links, 58 joints
Joints:
- joint HNP: origin xyz=0 0 0 rpy=0 -0 0 -> xyz=-0.0014665 0.0024526 0.0876725 rpy=0 -0 0
- joint HNR: origin xyz=-0.0014665 0.0024526 0.0876725 rpy=0 -0 0 -> xyz=0 0 0 rpy=0 -0 0
