Commit message: Manual update. Makes Hubo LIVE available for everyone.

File: data/hubo-urdf/model.urdf (robot description, URDF)
Before this commit: robot huboplus, 59 links, 58 joints
Links:
- removed link Body_LEP
- removed link Body_LKP
- removed link Body_REP
- removed link Body_RKP
- added link Body_LEB, mass 0.44094; collision mesh filename=./meshes/Body_LEB_col.dae; visual mesh filename=./meshes/Body_LEB_vis.dae
- added link Body_LKN, mass 1.80912; collision mesh filename=./meshes/Body_LKN_col.dae; visual mesh filename=./meshes/Body_LKN_vis.dae
- added link Body_REB, mass 0.44094; collision mesh filename=./meshes/Body_REB_col.dae; visual mesh filename=./meshes/Body_REB_vis.dae
- added link Body_RKN, mass 1.80912; collision mesh filename=./meshes/Body_RKN_col.dae; visual mesh filename=./meshes/Body_RKN_vis.dae
- link Body_Head: geometry collision mesh filename=./meshes/Body_Head.stl; visual mesh filename=./meshes/Body_Head.stl
- link leftIndexDistal: geometry collision mesh filename=./meshes/medial_distal.dae; visual mesh filename=./meshes/medial_distal.dae
- link leftIndexMedial: geometry collision mesh filename=./meshes/medial_distal.dae; visual mesh filename=./meshes/medial_distal.dae
- link leftIndexProximal: geometry collision mesh filename=./meshes/proximal.dae; visual mesh filename=./meshes/proximal.dae
- link leftMiddleDistal: geometry collision mesh filename=./meshes/medial_distal.dae; visual mesh filename=./meshes/medial_distal.dae
- link leftMiddleMedial: geometry collision mesh filename=./meshes/medial_distal.dae; visual mesh filename=./meshes/medial_distal.dae
- link leftMiddleProximal: geometry collision mesh filename=./meshes/proximal.dae; visual mesh filename=./meshes/proximal.dae
- link leftPinkyDistal: geometry collision mesh filename=./meshes/medial_distal.dae; visual mesh filename=./meshes/medial_distal.dae
- link leftPinkyMedial: geometry collision mesh filename=./meshes/medial_distal.dae; visual mesh filename=./meshes/medial_distal.dae
- link leftPinkyProximal: geometry collision mesh filename=./meshes/proximal.dae; visual mesh filename=./meshes/proximal.dae
- link leftRingDistal: geometry collision mesh filename=./meshes/medial_distal.dae; visual mesh filename=./meshes/medial_distal.dae
- link leftRingMedial: geometry collision mesh filename=./meshes/medial_distal.dae; visual mesh filename=./meshes/medial_distal.dae
- link leftRingProximal: geometry collision mesh filename=./meshes/proximal.dae; visual mesh filename=./meshes/proximal.dae
- link leftThumbDistal: geometry collision mesh filename=./meshes/medial_distal.dae; visual mesh filename=./meshes/medial_distal.dae
- link leftThumbMedial: geometry collision mesh filename=./meshes/medial_distal.dae; visual mesh filename=./meshes/medial_distal.dae
- link leftThumbProximal: geometry collision mesh filename=./meshes/proximal.dae; visual mesh filename=./meshes/proximal.dae
- link rightIndexDistal: geometry collision mesh filename=./meshes/medial_distal.dae; visual mesh filename=./meshes/medial_distal.dae
- link rightIndexMedial: geometry collision mesh filename=./meshes/medial_distal.dae; visual mesh filename=./meshes/medial_distal.dae
- link rightIndexProximal: geometry collision mesh filename=./meshes/proximal.dae; visual mesh filename=./meshes/proximal.dae
- link rightMiddleDistal: geometry collision mesh filename=./meshes/medial_distal.dae; visual mesh filename=./meshes/medial_distal.dae
- link rightMiddleMedial: geometry collision mesh filename=./meshes/medial_distal.dae; visual mesh filename=./meshes/medial_distal.dae
- link rightMiddleProximal: geometry collision mesh filename=./meshes/proximal.dae; visual mesh filename=./meshes/proximal.dae
- link rightPinkyDistal: geometry collision mesh filename=./meshes/medial_distal.dae; visual mesh filename=./meshes/medial_distal.dae
- link rightPinkyMedial: geometry collision mesh filename=./meshes/medial_distal.dae; visual mesh filename=./meshes/medial_distal.dae
- link rightPinkyProximal: geometry collision mesh filename=./meshes/proximal.dae; visual mesh filename=./meshes/proximal.dae
- link rightRingDistal: geometry collision mesh filename=./meshes/medial_distal.dae; visual mesh filename=./meshes/medial_distal.dae
- link rightRingMedial: geometry collision mesh filename=./meshes/medial_distal.dae; visual mesh filename=./meshes/medial_distal.dae
- link rightRingProximal: geometry collision mesh filename=./meshes/proximal.dae; visual mesh filename=./meshes/proximal.dae
- link rightThumbDistal: geometry collision mesh filename=./meshes/medial_distal.dae; visual mesh filename=./meshes/medial_distal.dae
- link rightThumbMedial: geometry collision mesh filename=./meshes/medial_distal.dae; visual mesh filename=./meshes/medial_distal.dae
- link rightThumbProximal: geometry collision mesh filename=./meshes/proximal.dae; visual mesh filename=./meshes/proximal.dae
Joints:
- removed joint LEP
- removed joint LKP
- removed joint REP
- removed joint RKP
- added joint LEB: type revolute, parent Body_LSY, child Body_LEB, origin xyz=0.0219936 -0.018 -0.157505 rpy=0 -0 0, axis 0 1 0, limit lower=-2.49582 upper=0.0698132 effort=10.0 velocity=1.0
- added joint LKN: type revolute, parent Body_LHP, child Body_LKN, origin xyz=0.000766364 -0.0445011 -0.280007 rpy=0 -0 0, axis 0 1 0, limit lower=-0.0698132 upper=2.60054 effort=10.0 velocity=1.0
- added joint REB: type revolute, parent Body_RSY, child Body_REB, origin xyz=0.0219936 0.018 -0.157505 rpy=0 -0 0, axis 0 1 0, limit lower=-2.49582 upper=0.0698132 effort=10.0 velocity=1.0
- added joint RKN: type revolute, parent Body_RHP, child Body_RKN, origin xyz=0.000766364 0.0445011 -0.280007 rpy=0 -0 0, axis 0 1 0, limit lower=-0.0698132 upper=2.60054 effort=10.0 velocity=1.0
- joint LAP: parent Body_LKP -> Body_LKN
- joint LWY: parent Body_LEP -> Body_LEB
- joint RAP: parent Body_RKP -> Body_RKN
- joint RWY: parent Body_REP -> Body_REB

Commit message: Updated webpage with new STL BufferGeometry.

File: data/hubo-urdf/model.urdf (robot description, URDF)
Before this commit: robot huboplus, 59 links, 58 joints
Links:
- link Body_Hip: geometry collision mesh filename=./meshes/Body_Hip.stl; visual mesh filename=./meshes/Body_Hip_vis.dae
- link Body_LAP: geometry collision mesh filename=./meshes/Body_LAP.stl; visual mesh filename=./meshes/Body_LAP.stl
- link Body_LAR: geometry collision mesh filename=./meshes/Body_LAR.stl; visual mesh filename=./meshes/Body_LAR.stl
- link Body_LEB: geometry collision mesh filename=./meshes/Body_LEB.stl; visual mesh filename=./meshes/Body_LEB.stl
- link Body_LHP: geometry collision mesh filename=./meshes/Body_LHP.stl; visual mesh filename=./meshes/Body_LHP.stl
- link Body_LHR: geometry collision mesh filename=./meshes/Body_LHR.stl; visual mesh filename=./meshes/Body_LHR.stl
- link Body_LHY: geometry collision mesh filename=./meshes/Body_LHY.stl; visual mesh filename=./meshes/Body_LHY.stl
- link Body_LKN: geometry collision mesh filename=./meshes/Body_LKN.stl; visual mesh filename=./meshes/Body_LKN_vis.dae
- link Body_LSP: geometry collision mesh filename=./meshes/Body_LSP.stl; visual mesh filename=./meshes/Body_LSP_vis.dae
- link Body_LSR: geometry collision mesh filename=./meshes/Body_LSR.stl; visual mesh filename=./meshes/Body_LSR_vis.dae
- link Body_LSY: geometry collision mesh filename=./meshes/Body_LSY.stl; visual mesh filename=./meshes/Body_LSY_vis.dae
- link Body_LWP: geometry collision mesh filename=./meshes/Body_LWP.stl; visual mesh filename=./meshes/Body_LWP_vis.dae
- link Body_LWY: geometry collision mesh filename=./meshes/Body_LWY.stl; visual mesh filename=./meshes/Body_LWY_vis.dae
- link Body_Neck: geometry collision mesh filename=./meshes/Body_Neck.stl
- link Body_RAP: geometry collision mesh filename=./meshes/Body_RAP.stl; visual mesh filename=./meshes/Body_RAP_vis.dae
- link Body_RAR: geometry collision mesh filename=./meshes/Body_RAR.stl; visual mesh filename=./meshes/Body_RAR_vis.dae
- link Body_REB: geometry collision mesh filename=./meshes/Body_REB.stl; visual mesh filename=./meshes/Body_REB_vis.dae
- link Body_RHP: geometry collision mesh filename=./meshes/Body_RHP.stl; visual mesh filename=./meshes/Body_RHP_vis.dae
- link Body_RHR: geometry collision mesh filename=./meshes/Body_RHR.stl; visual mesh filename=./meshes/Body_RHR_vis.dae
- link Body_RHY: geometry collision mesh filename=./meshes/Body_RHY.stl; visual mesh filename=./meshes/Body_RHY_vis.dae
- link Body_RKN: geometry collision mesh filename=./meshes/Body_RKN.stl; visual mesh filename=./meshes/Body_RKN_vis.dae
- link Body_RSP: geometry collision mesh filename=./meshes/Body_RSP.stl; visual mesh filename=./meshes/Body_RSP_vis.dae
- link Body_RSR: geometry collision mesh filename=./meshes/Body_RSR.stl; visual mesh filename=./meshes/Body_RSR_vis.dae
- link Body_RSY: geometry collision mesh filename=./meshes/Body_RSY.stl; visual mesh filename=./meshes/Body_RSY_vis.dae
- link Body_RWP: geometry collision mesh filename=./meshes/Body_RWP.stl; visual mesh filename=./meshes/Body_RWP_vis.dae
- link Body_RWY: geometry collision mesh filename=./meshes/Body_RWY.stl; visual mesh filename=./meshes/Body_RWY_vis.dae
- link Body_Torso: geometry collision mesh filename=./meshes/Body_Torso.stl; visual mesh filename=./meshes/Body_Torso_vis.dae
- link leftIndexDistal: geometry collision mesh filename=./meshes/medial_distal.stl; visual mesh filename=./meshes/medial_distal.stl
- link leftIndexMedial: geometry collision mesh filename=./meshes/medial_distal.stl; visual mesh filename=./meshes/medial_distal.stl
- link leftIndexProximal: geometry collision mesh filename=./meshes/proximal.stl; visual mesh filename=./meshes/proximal.stl
- link leftMiddleDistal: geometry collision mesh filename=./meshes/medial_distal.stl; visual mesh filename=./meshes/medial_distal.stl
- link leftMiddleMedial: geometry collision mesh filename=./meshes/medial_distal.stl; visual mesh filename=./meshes/medial_distal.stl
- link leftMiddleProximal: geometry collision mesh filename=./meshes/proximal.stl; visual mesh filename=./meshes/proximal.stl
- link leftPinkyDistal: geometry collision mesh filename=./meshes/medial_distal.stl; visual mesh filename=./meshes/medial_distal.stl
- link leftPinkyMedial: geometry collision mesh filename=./meshes/medial_distal.stl; visual mesh filename=./meshes/medial_distal.stl
- link leftPinkyProximal: geometry collision mesh filename=./meshes/proximal.stl; visual mesh filename=./meshes/proximal.stl
- link leftRingDistal: geometry collision mesh filename=./meshes/medial_distal.stl; visual mesh filename=./meshes/medial_distal.stl
- link leftRingMedial: geometry collision mesh filename=./meshes/medial_distal.stl; visual mesh filename=./meshes/medial_distal.stl
- link leftRingProximal: geometry collision mesh filename=./meshes/proximal.stl; visual mesh filename=./meshes/proximal.stl
- link leftThumbDistal: geometry collision mesh filename=./meshes/medial_distal.stl; visual mesh filename=./meshes/medial_distal.stl
- link leftThumbMedial: geometry collision mesh filename=./meshes/medial_distal.stl; visual mesh filename=./meshes/medial_distal.stl
- link leftThumbProximal: geometry collision mesh filename=./meshes/proximal.stl; visual mesh filename=./meshes/proximal.stl
- link rightIndexDistal: geometry collision mesh filename=./meshes/medial_distal.stl; visual mesh filename=./meshes/medial_distal.stl
- link rightIndexMedial: geometry collision mesh filename=./meshes/medial_distal.stl; visual mesh filename=./meshes/medial_distal.stl
- link rightIndexProximal: geometry collision mesh filename=./meshes/proximal.stl; visual mesh filename=./meshes/proximal.stl
- link rightMiddleDistal: geometry collision mesh filename=./meshes/medial_distal.stl; visual mesh filename=./meshes/medial_distal.stl
- link rightMiddleMedial: geometry collision mesh filename=./meshes/medial_distal.stl; visual mesh filename=./meshes/medial_distal.stl
- link rightMiddleProximal: geometry collision mesh filename=./meshes/proximal.stl; visual mesh filename=./meshes/proximal.stl
- link rightPinkyDistal: geometry collision mesh filename=./meshes/medial_distal.stl; visual mesh filename=./meshes/medial_distal.stl
- link rightPinkyMedial: geometry collision mesh filename=./meshes/medial_distal.stl; visual mesh filename=./meshes/medial_distal.stl
- link rightPinkyProximal: geometry collision mesh filename=./meshes/proximal.stl; visual mesh filename=./meshes/proximal.stl
- link rightRingDistal: geometry collision mesh filename=./meshes/medial_distal.stl; visual mesh filename=./meshes/medial_distal.stl
- link rightRingMedial: geometry collision mesh filename=./meshes/medial_distal.stl; visual mesh filename=./meshes/medial_distal.stl
- link rightRingProximal: geometry collision mesh filename=./meshes/proximal.stl; visual mesh filename=./meshes/proximal.stl
- link rightThumbDistal: geometry collision mesh filename=./meshes/medial_distal.stl; visual mesh filename=./meshes/medial_distal.stl
- link rightThumbMedial: geometry collision mesh filename=./meshes/medial_distal.stl; visual mesh filename=./meshes/medial_distal.stl
- link rightThumbProximal: geometry collision mesh filename=./meshes/proximal.stl; visual mesh filename=./meshes/proximal.stl
